File: usb-type-c-hhkb.kicad_pcb (KiCad board)
At the start: 2 copper layers, 12.9 x 12.4 mm, 7 parts, among them J1 USB_TYPE_C, P1 GND, P2 D+, P3 D-, P4 VCC

Commit message: Rev2
Parts:
- J1: footprint usb-type-c:JAE-DX07S024JJ2-oshpark -> usb-type-c:JAE-DX07S024JJ2-oshpark-cutpads
- moved R1 0.06 mm to (148.7, 91.4)
Routing:
- net GND: track 21.4 -> 45.7 mm, vias 1 -> 2
- net /CC2: track 9.60 -> 7.25 mm
- net VCC: track 12.1 -> 10.6 mm, vias 0 -> 2
- net /USB_D-: track 7.89 -> 6.42 mm
- added copper zone on B.Cu, net GND
- added copper zone on F.Cu, net GND
Other:
- outline, holes or cut-outs redrawn
- board text added: "R2"
- board text removed: "R1"

Commit message: Rev3
Routing:
- net GND: track 45.7 -> 65.6 mm
Other:
- board text added: "R3"
- board text removed: "R2"
